File: Connectors.kicad_sch (KiCad schematic)
At the start: 2 parts, among them J2 Conn_01x15, J3 Conn_01x15

Commit message: Added Footprints to the Symbols
Parts:
- J2, J3: footprint (none) -> Connector_PinHeader_2.54mm:PinHeader_1x15_P2.54mm_Vertical
Changed lines of the file:
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@@
 			)
 		)
-		(property "Footprint" ""
+		(property "Footprint" "Connector_PinHeader_2.54mm:PinHeader_1x15_P2.54mm_Vertical"
 			(at 110.998 87.63 0)
 			(effects
@@
 			)
 		)
-		(property "Footprint" ""
+		(property "Footprint" "Connector_PinHeader_2.54mm:PinHeader_1x15_P2.54mm_Vertical"
 			(at 163.83 87.376 0)
 			(effects
